File: smartCurtains_sch.sch (KiCad schematic (older format))
At the start: 42 parts, among them J1 Conn_01x02, J2 , J3 Conn_01x06, K1 IM44, Q1 2N7002, Q2 MMBT2222A, SW1 SW_665, U1 LM25011, U2 LM1117-3.3, U3 ESP32-PICO-D4

Commit message: update
Parts:
- added D3: LED, symbol Device:LED
- added R13: 10k, symbol Device:R_Small
- added R7: 470R, symbol Device:R_Small
- J3: value Conn_01x06 -> (none)
- R1: value R -> 10k
- R14: value 0R(5%) -> 10k
Connections:
- net +3V3: now also C13.1, C14.1, R14.2, U3.43 (VDDA), U3.46 (VDDA), R13.2, R7.1
- net EN: now also C15.1, R12.2, R14.1, SW1.2; no longer R14.2
- net GND: now also D3.1 (K)
- net GPIO0: now also R13.1
- net GPIO4: now reaches U3.24 (IO4/A2_0/T0)
- net GPIO4: now also D3.2 (A), R7.2
- no-connect marks 22 -> 21
Other:
- moved on the sheet: J3
Changed lines of the file:
@@
 $EndComp
 Wire Wire Line
-	2650 750  2650 1600
+	2650 750  2650 950
 Wire Wire Line
 	3250 1600 3250 950
 Wire Wire Line
-	3250 950  2100 950
+	3250 950  2650 950
 Connection ~ 2100 950
 Wire Wire Line
@@
 Encoder
 $Comp
-L Switches_Button:SW_665 SW1
-U 1 1 5B8095CE
-P 4950 4000
-F 0 "SW1" H 4950 4193 50  0000 C CNN
-F 1 "SW_665" H 4950 3940 50  0001 C CNN
-F 2 "Button_Switch_THT:SW_PUSH_6mm_H5mm" H 4950 4200 50  0001 C CNN
-F 3 "https://www.mouser.vn/datasheet/2/15/SKHH-1370651.pdf" H 4950 4200 50  0001 C CNN
-F 4 "SKHHAKA010" H 5100 4200 50  0001 C CNN "manf#"
-	1    4950 4000
-	1    0    0    -1
-$EndComp
-$Comp
 L power:GND #PWR0123
 U 1 1 5B814091
@@
 	0    -1   -1   0
 $EndComp
-Wire Wire Line
-	4300 2950 4500 2950
 $Comp
 L Connector_Generic:Conn_01x06 J3
 U 1 1 5B7C38C3
-P 1400 3500
-F 0 "J3" H 1480 3492 50  0000 L CNN
-F 1 "Conn_01x06" H 1480 3401 50  0000 L CNN
-F 2 "" H 1400 3500 50  0001 C CNN
-F 3 "~" H 1400 3500 50  0001 C CNN
-	1    1400 3500
+P 1500 2550
+F 0 "J3" H 1580 2542 50  0000 L CNN
+F 1 " " H 1580 2451 50  0000 L CNN
+F 2 "" H 1500 2550 50  0001 C CNN
+F 3 "~" H 1500 2550 50  0001 C CNN
+	1    1500 2550
 	1    0    0    -1
 $EndComp
@@
 L power:+3.3V #PWR0130
 U 1 1 5B7C987B
-P 1050 3050
-F 0 "#PWR0130" H 1050 2900 50  0001 C CNN
-F 1 "+3.3V" H 1065 3223 50  0000 C CNN
-F 2 "" H 1050 3050 50  0001 C CNN
-F 3 "" H 1050 3050 50  0001 C CNN
-	1    1050 3050
-	1    0    0    -1
-$EndComp
-Wire Wire Line
-	1200 3300 1050 3300
-Wire Wire Line
-	1050 3300 1050 3050
-Text GLabel 1050 3500 0    50   Input ~ 0
+P 1150 2100
+F 0 "#PWR0130" H 1150 1950 50  0001 C CNN
+F 1 "+3.3V" H 1165 2273 50  0000 C CNN
+F 2 "" H 1150 2100 50  0001 C CNN
+F 3 "" H 1150 2100 50  0001 C CNN
+	1    1150 2100
+	1    0    0    -1
+$EndComp
+Wire Wire Line
+	1300 2350 1150 2350
+Wire Wire Line
+	1150 2350 1150 2100
+Text GLabel 1150 2550 0    50   Input ~ 0
 Rx
-Text GLabel 1050 3600 0    50   Input ~ 0
+Text GLabel 1150 2650 0    50   Input ~ 0
 Tx
-Text GLabel 1050 3700 0    50   Input ~ 0
+Text GLabel 1150 2750 0    50   Input ~ 0
 GPIO0
-Text GLabel 1050 3800 0    50   Input ~ 0
+Text GLabel 1150 2850 0    50   Input ~ 0
 EN
 Wire Wire Line
-	1200 3500 1050 3500
-Wire Wire Line
-	1200 3600 1050 3600
-Wire Wire Line
-	1050 3700 1200 3700
-Wire Wire Line
-	1050 3800 1200 3800
-Wire Wire Line
-	1200 3400 700  3400
-Wire Wire Line
-	700  3400 700  4100
+	1300 2550 1150 2550
+Wire Wire Line
+	1300 2650 1150 2650
+Wire Wire Line
+	1150 2750 1300 2750
+Wire Wire Line
+	1150 2850 1300 2850
+Wire Wire Line
+	1300 2450 800  2450
+Wire Wire Line
+	800  2450 800  3150
 Text GLabel 2950 1500 1    50   Input ~ 0
 Rx
@@
 NoConn ~ 4300 3050
 NoConn ~ 4300 3150
-NoConn ~ 2650 3800
 NoConn ~ 2850 3800
 NoConn ~ 2950 3800
@@
 Text GLabel 2750 3950 3    50   Input ~ 0
 GPIO0
-Wire Wire Line
-	2750 3800 2750 3950
 $Comp
 L power:GND #PWR0111
@@
 L power:GND #PWR0106
 U 1 1 5B9561F0
-P 700 4100
-F 0 "#PWR0106" H 700 3850 50  0001 C CNN
-F 1 "GND" H 705 3927 50  0000 C CNN
-F 2 "" H 700 4100 50  0001 C CNN
-F 3 "" H 700 4100 50  0001 C CNN
-	1    700  4100
+P 800 3150
+F 0 "#PWR0106" H 800 2900 50  0001 C CNN
+F 1 "GND" H 805 2977 50  0000 C CNN
+F 2 "" H 800 3150 50  0001 C CNN
+F 3 "" H 800 3150 50  0001 C CNN
+	1    800  3150
 	1    0    0    -1
 $EndComp
@@
 Wire Wire Line
 	2900 4650 2900 4550
-Wire Wire Line
-	3150 3800 3150 4650
 Wire Wire Line
 	3950 1300 4100 1300
@@
 P 1050 5700
 F 0 "R1" V 854 5700 50  0000 C CNN
-F 1 "R" V 945 5700 50  0000 C CNN
+F 1 "10k" V 945 5700 50  0000 C CNN
 F 2 "" H 1050 5700 50  0001 C CNN
 F 3 "~" H 1050 5700 50  0001 C CNN
@@
 Wire Wire Line
 	5400 3800 5400 4000
-$Comp
-L Device:R_Small R14
-U 1 1 5B8351F3
-P 5750 4000
-F 0 "R14" V 5950 3950 50  0000 L CNN
-F 1 "0R(5%)" V 5850 3850 50  0000 L CNN
-F 2 "" H 5750 4000 50  0001 C CNN
-F 3 "~" H 5750 4000 50  0001 C CNN
-	1    5750 4000
-	0    -1   -1   0
-$EndComp
-Wire Wire Line
-	5400 4000 5650 4000
-Wire Wire Line
-	5850 4000 6200 4000
 Wire Wire Line
 	4050 5700 4200 5700
@@
 	1    0    0    -1
 $EndComp
-$Comp
-L power:+3.3V #PWR0136
-U 1 1 5B908DCA
-P 6350 5850
-F 0 "#PWR0136" H 6350 5700 50  0001 C CNN
-F 1 "+3.3V" H 6365 6023 50  0000 C CNN
-F 2 "" H 6350 5850 50  0001 C CNN
-F 3 "" H 6350 5850 50  0001 C CNN
-	1    6350 5850
-	1    0    0    -1
-$EndComp
-Wire Wire Line
-	6200 6100 6350 6100
-Wire Wire Line
-	6350 6100 6350 6200
-Wire Wire Line
-	6350 5850 6350 6100
-Connection ~ 6350 6100
 Wire Wire Line
 	6350 6400 6350 6550
@@
 Wire Wire Line
 	5400 5850 5400 6100
-$Comp
-L power:PWR_FLAG #FLG0104
-U 1 1 5B999209
-P 2600 7100
-F 0 "#FLG0104" H 2600 7175 50  0001 C CNN
-F 1 "PWR_FLAG" H 2600 7274 50  0000 C CNN
-F 2 "" H 2600 7100 50  0001 C CNN
-F 3 "~" H 2600 7100 50  0001 C CNN
-	1    2600 7100
-	1    0    0    -1
-$EndComp
-Wire Wire Line
-	2600 7150 2600 7100
 Text Notes 2950 7700 0    79   ~ 16
 POWER
@@
 Wire Bus Line
 	9400 4050 11250 4050
+Wire Wire Line
+	5400 4000 6200 4000
+Wire Wire Line
+	3150 3800 3150 4650
+$Comp
+L power:+3.3V #PWR0122
+U 1 1 5B7AA50A
+P 4650 750
+F 0 "#PWR0122" H 4650 600 50  0001 C CNN
+F 1 "+3.3V" H 4665 923 50  0000 C CNN
+F 2 "" H 4650 750 50  0001 C CNN
+F 3 "" H 4650 750 50  0001 C CNN
+	1    4650 750
+	1    0    0    -1
+$EndComp
+Text GLabel 5250 900  2    50   Input ~ 0
+GPIO0
+Text GLabel 5250 1200 2    50   Input ~ 0
+EN
+Wire Wire Line
+	4650 750  4650 900
+$Comp
+L Device:R_Small R13
+U 1 1 5B7C9BC5
+P 4950 900
+F 0 "R13" V 4754 900 50  0000 C CNN
+F 1 "10k" V 4845 900 50  0000 C CNN
+F 2 "" H 4950 900 50  0001 C CNN
+F 3 "~" H 4950 900 50  0001 C CNN
+	1    4950 900
+	0    1    1    0
+$EndComp
+$Comp
+L Device:R_Small R14
+U 1 1 5B7C9C74
+P 4950 1200
+F 0 "R14" V 4754 1200 50  0000 C CNN
+F 1 "10k" V 4845 1200 50  0000 C CNN
+F 2 "" H 4950 1200 50  0001 C CNN
+F 3 "~" H 4950 1200 50  0001 C CNN
+	1    4950 1200
+	0    1    1    0
+$EndComp
+Wire Wire Line
+	5250 900  5050 900
+Wire Wire Line
+	4850 900  4650 900
+Connection ~ 4650 900
+Wire Wire Line
+	4650 900  4650 1200
+Wire Wire Line
+	4850 1200 4650 1200
+Wire Wire Line
+	5250 1200 5050 1200
+Wire Wire Line
+	2750 3800 2750 3950
+$Comp
+L Switches_Button:SW_665 SW1
+U 1 1 5B8095CE
+P 4950 4000
+F 0 "SW1" H 4950 4193 50  0000 C CNN
+F 1 "SW_665" H 4950 3940 50  0001 C CNN
+F 2 "Button_Switch_THT:SW_PUSH_6mm_H5mm" H 4950 4200 50  0001 C CNN
+F 3 "https://www.mouser.vn/datasheet/2/15/SKHH-1370651.pdf" H 4950 4200 50  0001 C CNN
+F 4 "SKHHAKA010" H 5100 4200 50  0001 C CNN "manf#"
+	1    4950 4000
+	1    0    0    -1
+$EndComp
+Wire Wire Line
+	4300 2950 4500 2950
+$Comp
+L power:+3.3V #PWR0140
+U 1 1 5B81E083
+P 1000 3650
+F 0 "#PWR0140" H 1000 3500 50  0001 C CNN
+F 1 "+3.3V" H 1015 3823 50  0000 C CNN
+F 2 "" H 1000 3650 50  0001 C CNN
+F 3 "" H 1000 3650 50  0001 C CNN
+	1    1000 3650
+	1    0    0    -1
+$EndComp
+$Comp
+L Device:R_Small R7
+U 1 1 5B81E12D
+P 1000 3900
+F 0 "R7" H 1059 3946 50  0000 L CNN
+F 1 "470R" H 1059 3855 50  0000 L CNN
+F 2 "" H 1000 3900 50  0001 C CNN
+F 3 "~" H 1000 3900 50  0001 C CNN
+	1    1000 3900
+	1    0    0    -1
+$EndComp
+$Comp
+L power:GND #PWR0141
+U 1 1 5B81E1F5
+P 1000 4700
+F 0 "#PWR0141" H 1000 4450 50  0001 C CNN
+F 1 "GND" H 1005 4527 50  0000 C CNN
+F 2 "" H 1000 4700 50  0001 C CNN
+F 3 "" H 1000 4700 50  0001 C CNN
+	1    1000 4700
+	1    0    0    -1
+$EndComp
+$Comp
+L Device:LED D3
+U 1 1 5B81E2B0
+P 1000 4400
+F 0 "D3" V 1038 4283 50  0000 R CNN
+F 1 "LED" V 947 4283 50  0000 R CNN
+F 2 "" H 1000 4400 50  0001 C CNN
+F 3 "~" H 1000 4400 50  0001 C CNN
+	1    1000 4400
+	0    -1   -1   0
+$EndComp
+Wire Wire Line
+	1000 3650 1000 3800
+Wire Wire Line
+	1000 4000 1000 4100
+Wire Wire Line
+	1000 4550 1000 4700
+Text GLabel 1350 4100 2    50   Input ~ 0
+GPIO4
+Wire Wire Line
+	1350 4100 1000 4100
+Connection ~ 1000 4100
+Wire Wire Line
+	1000 4100 1000 4250
+Text GLabel 2650 3950 3    50   Input ~ 0
+GPIO4
+Wire Wire Line
+	2650 3800 2650 3950
+Wire Wire Line
+	6200 6100 6350 6100
+Wire Wire Line
+	6350 6100 6350 6200
+$Comp
+L power:+3.3V #PWR0136
+U 1 1 5B908DCA
+P 6350 5850
+F 0 "#PWR0136" H 6350 5700 50  0001 C CNN
+F 1 "+3.3V" H 6365 6023 50  0000 C CNN
+F 2 "" H 6350 5850 50  0001 C CNN
+F 3 "" H 6350 5850 50  0001 C CNN
+	1    6350 5850
+	1    0    0    -1
+$EndComp
+Connection ~ 6350 6100
+Wire Wire Line
+	6350 5850 6350 6100
+$Comp
+L power:PWR_FLAG #FLG0101
+U 1 1 5B880EB3
+P 2600 7050
+F 0 "#FLG0101" H 2600 7125 50  0001 C CNN
+F 1 "PWR_FLAG" H 2600 7224 50  0000 C CNN
+F 2 "" H 2600 7050 50  0001 C CNN
+F 3 "~" H 2600 7050 50  0001 C CNN
+	1    2600 7050
+	1    0    0    -1
+$EndComp
+Wire Wire Line
+	2600 7050 2600 7150
+Connection ~ 2650 950
+Wire Wire Line
+	2650 950  2650 1600
+Wire Wire Line
+	2650 950  2100 950
 $EndSCHEMATC
